Commit message: add a simulation script that uses pinocchio

File: robot/hardware/furuta.urdf (robot description, URDF)
Before this commit: robot furuta_pendulum, 5 links, 4 joints
Links:
- link arm1: geometry visual cylinder length=0.2 radius=0.005
- link arm2: geometry visual cylinder length=0.1 radius=0.005
- link arm_mount: mass 0.0 -> 0.1; geometry visual mesh filename=37d_arm.stl scale=0.001 0.001 0.001
- link base_link: geometry visual mesh filename=37d_motor_mount.stl scale=0.001 0.001 0.001
