Commit message: update urdf to have pendulum down

File: robot/hardware/URDF/robot.urdf (robot description, URDF)
Before this commit: robot onshape, 3 links, 2 joints
Joints:
- joint arm: origin xyz=-0.0040000000000000139611 -1.3010426069826053208e-18 0.0091500000000000053513 rpy=-1.570796326794896558 8.7284454278903452765e-14 1.5707963267948801267 -> xyz=-0.0040000000000000139611 -1.3010426069826053208e-18 0.0091500000000000053513 rpy=-1.570796326794896558 3.14159265359 1.5707963267948801267
