Commit message: adapt names in urdf

File: robot/hardware/v2/robot.urdf (robot description, URDF)
Before this commit: robot onshape, 3 links, 2 joints
Links:
- link arm: geometry visual mesh filename=package:///37d_arm.stl; visual mesh filename=package:///8x22x7_bearing.stl
- link base_link: geometry visual mesh filename=package:///37d_motor_mount.stl

Commit message: merge STLs

File: robot/hardware/v2/robot.urdf (robot description, URDF)
Before this commit: robot onshape, 3 links, 2 joints
Links:
- link arm: geometry visual mesh filename=package:///arm_visual.stl
- link base_link: geometry visual mesh filename=package:///base_link_visual.stl
- link pendulum: mass 0.030800000000000004458 -> 0.030800000000000000988; geometry visual mesh filename=package:///pendulum_visual.stl
Joints:
- joint arm: origin xyz=-0.0040000000000000139611 -1.3010426069826053208e-18 0.0091500000000000053513 rpy=-1.570796326794896558 3.14159265359 1.5707963267948801267 -> xyz=-0.0040000000000000139611 -1.3010426069826053208e-18 0.0091500000000000053513 rpy=-1.570796326794896558 3.141592653589793 1.5707963267948801267

Commit message: new urdf with mass closer to reality

File: robot/hardware/v2/robot.urdf (robot description, URDF)
Before this commit: robot penduli, 3 links, 2 joints
Links:
- link arm: mass 0.05050000000000000322 -> 0.053300000000000000155
- link pendulum: mass 0.030800000000000000988 -> 0.045800000000000007372

Commit message: reverse pendulum rotation axis

File: robot/hardware/v2/robot.urdf (robot description, URDF)
Before this commit: robot penduli, 3 links, 2 joints
Links:
- link arm: mass 0.053300000000000000155 -> 0.053299999999999979339
- link pendulum: mass 0.045800000000000007372 -> 0.045800000000000000433
Joints:
- joint arm: origin xyz=-0.0040000000000000139611 -1.3010426069826053208e-18 0.0091500000000000053513 rpy=-1.570796326794896558 3.141592653589793 1.5707963267948801267 -> xyz=0.0039999999999999723277 0 0.0091499999999999914735 rpy=1.570796326794896558 -5.9231157207999756293e-08 1.570796326794896558
- joint base_link: origin xyz=0.0031935242862665912632 -0.0071650681287528461896 0.090081326273058190401 rpy=3.0839735524825034295e-14 3.011479954295665724e-15 1.5707963267948303887 -> xyz=0.01627551605615560476 -0.014200560520388399999 0.072862520335433791918 rpy=1.6199343425107188831e-09 1.2085681117354552082e-07 1.5707963785076977103

Commit message: update urdf for better viz -> no dynamics changes

File: robot/hardware/v2/robot.urdf (robot description, URDF)
Before this commit: robot penduli, 3 links, 2 joints
Joints:
- joint arm: origin xyz=0.0039999999999999723277 0 0.0091499999999999914735 rpy=1.570796326794896558 -5.9231157207999756293e-08 1.570796326794896558 -> xyz=0.0039999999999999723277 0 0.0091499999999999914735 rpy=1.57079632679489661923 0.0 1.57079632679489661923
- joint base_link: origin xyz=0.01627551605615560476 -0.014200560520388399999 0.072862520335433791918 rpy=1.6199343425107188831e-09 1.2085681117354552082e-07 1.5707963785076977103 -> xyz=0.0 0.0 0.085 rpy=0.0 0.0 0.0
